File: gimbal.kicad_pcb (KiCad board)
At the start: 2 copper layers, 103 parts, among them J1 USB_C_Receptacle_USB2.0_16P, J2 JTAG, J3 Pitch, J4 Roll, J5 Yaw, J6 IMU_Payload, J7 Power_9V, J8 UART3, J9 UART2, SW1 SW_Push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

Commit message: ...
Parts:
- SW1: value SW_Push -> Reset; footprint Button_Switch_THT:SW_PUSH_6mm_H5mm -> Button_Switch_SMD:SW_SPST_B3U-1000P
- SW2: value SW_Push -> Boot; footprint Button_Switch_THT:SW_PUSH_6mm_H5mm -> Button_Switch_SMD:SW_SPST_B3U-1000P
- Y1: footprint Crystal:Crystal_SMD_0603-2Pin_6.0x3.5mm_HandSoldering -> Crystal:Crystal_SMD_2012-2Pin_2.0x1.2mm_HandSoldering
- Y2: footprint Crystal:Crystal_SMD_3225-4Pin_3.2x2.5mm -> Crystal:Crystal_SMD_2016-4Pin_2.0x1.6mm
- moved J7 185.5 mm to (176.0, 130.8)
- moved R5 150.1 mm to (126.8, 156.0), turned to 90 degrees
- moved R4 149.6 mm to (127.5, 156.0), turned to -90 degrees
- moved R7 147.7 mm to (128.8, 156.0), turned to -90 degrees
- moved R6 145.0 mm to (131.8, 156.0), turned to -90 degrees
- moved D2 143.3 mm to (136.2, 153.2)
- moved C9 141.2 mm to (126.0, 156.0), turned to 90 degrees
- moved J1 140.9 mm to (130.0, 161.8)
- moved R23 134.7 mm to (157.7, 131.3)
- moved R26 134.5 mm to (156.5, 133.3), turned to -90 degrees
- moved JP2 134.3 mm to (122.5, 154.2), turned to -90 degrees
- moved R24 133.6 mm to (157.7, 130.6), turned to 180 degrees
- moved R27 132.9 mm to (157.7, 133.8), turned to 180 degrees
- moved R28 132.8 mm to (157.7, 135.3), turned to 180 degrees
- moved R29 131.8 mm to (157.7, 134.6), turned to 180 degrees
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