File: gimbal.kicad_pcb (KiCad board)
At the start: 2 copper layers, 103 parts, among them J1 USB_C_Receptacle_USB2.0_16P, J2 JTAG, J3 Pitch, J4 Roll, J5 Yaw, J6 IMU_Payload, J7 Power_9V, J8 UART3, J9 UART2, SW1 Reset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

Commit message: ...
Parts:
- moved J9 113.4 mm to (206.8, 71.4), turned to 90 degrees
- moved J6 110.5 mm to (206.8, 96.4), turned to 90 degrees
- moved J8 109.5 mm to (206.8, 83.8), turned to 90 degrees
- moved C22 95.3 mm to (202.4, 108.9)
- moved D5 95.3 mm to (201.2, 103.0)
- moved R14 95.3 mm to (199.4, 102.6)
- moved R15 95.3 mm to (202.4, 106.4)
- moved SW1 95.3 mm to (200.2, 107.5)
- moved J2 88.0 mm to (184.3, 78.4), turned to 90 degrees
- moved C8 77.8 mm to (188.3, 81.6), turned to 90 degrees
- moved Y2 77.7 mm to (188.2, 83.9)
- moved C9 77.5 mm to (187.2, 99.4)
- moved J1 77.5 mm to (191.2, 105.7)
- moved R4 77.5 mm to (189.2, 99.4)
- moved R5 77.5 mm to (188.2, 99.4)
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Routing:
- net GND: track 19.5 -> 59.1 mm
- net VCC: track 7.70 -> 26.5 mm
- net Net-(D8-K): track 0.00 -> 12.1 mm
- net Net-(U7-FB): track 0.00 -> 6.68 mm
- net /Pitch1: track 0.00 -> 6.65 mm
- net /Roll1: track 0.00 -> 6.61 mm
- net /Roll3: track 0.00 -> 6.53 mm
- net /Pitch3: track 0.00 -> 6.51 mm
- net /PA8_SCL: track 1.48 -> 7.78 mm
- net /Pitch2: track 0.00 -> 6.07 mm
- net /Roll2: track 0.00 -> 6.05 mm
- net /FLT_DRV1: track 0.00 -> 5.41 mm
- net /FLT_DRV2: track 0.00 -> 5.31 mm
- net /PC11_SDA: track 1.50 -> 6.19 mm
- net Net-(U7-EN): track 0.00 -> 4.30 mm
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
Commit message: ...
Parts:
- moved D7 21.8 mm to (155.1, 100.3)
- moved JP6 21.8 mm to (154.9, 97.2)
- moved R22 21.8 mm to (155.8, 102.3)
- moved JP5 21.3 mm to (155.2, 85.4)
- moved D6 21.3 mm to (155.4, 88.5)
- moved R19 21.3 mm to (156.2, 90.5)
- moved D1 21.1 mm to (155.6, 76.0)
- moved JP4 21.1 mm to (155.4, 72.8)
- moved R1 21.1 mm to (156.4, 78.0)
- moved D4 1.80 mm to (183.2, 103.0)
- moved R13 1.80 mm to (183.3, 100.8)
- moved C5 0.68 mm to (193.5, 81.4)
- moved C6 0.68 mm to (191.5, 81.4)
- moved Y1 0.68 mm to (192.4, 83.2)
- moved Y2 0.68 mm to (188.8, 84.2)
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Connections:
- U5 pad 22: /PC6 -> /PB15
- U5 pad 24: /PC6 -> /PB15
- U5 pad 26: /PC6 -> /PB15
- U6 pad 22: /PC6 -> /PB14
- U6 pad 24: /PC6 -> /PB14
- U6 pad 26: /PC6 -> /PB14
Routing:
- net GND: track 59.1 -> 88.8 mm, vias 0 -> 15
- net /PA0: track 0.00 -> 27.1 mm, vias 0 -> 2
- net /PA1: track 0.00 -> 25.8 mm, vias 0 -> 2
- net /PA2: track 0.00 -> 24.9 mm, vias 0 -> 2
- net /PB0: track 0.00 -> 14.9 mm, vias 0 -> 1
- net /PA4: track 0.00 -> 14.9 mm, vias 0 -> 1
- net /PB15: track 0.00 -> 6.85 mm, vias 0 -> 4
- net /FLT_DRV3: track 5.62 -> 0.04 mm
- net /FLT_DRV1: track 5.41 -> 0.00 mm
- net /PB14: track 0.00 -> 5.28 mm, vias 0 -> 3
- net /FLT_DRV2: track 5.31 -> 0.04 mm
- net /PC6: track 0.00 -> 5.13 mm, vias 0 -> 3
- net /PB4: track 0.00 -> 3.61 mm, vias 0 -> 2
- net /PB6: track 0.00 -> 3.56 mm, vias 0 -> 1
- net /PB9: track 0.00 -> 3.56 mm, vias 0 -> 1
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
Commit message: ...
Parts:
- removed D4: LED, LED_SMD:LED_0603_1608Metric
- removed R13: 5.1k, Resistor_SMD:R_0201_0603Metric_Pad0.64x0.40mm_HandSolder
- moved C23 133.9 mm to (59.4, 91.9), turned to 0 degrees
- moved D5 133.7 mm to (73.7, 62.6), turned to -90 degrees
- moved R14 131.1 mm to (73.7, 65.2), turned to 180 degrees
- moved D2 130.2 mm to (67.6, 97.8)
- moved C9 128.6 mm to (58.6, 100.1)
- moved R4 128.6 mm to (60.6, 100.1)
- moved R5 128.6 mm to (59.6, 100.1)
- moved R7 128.6 mm to (61.6, 100.1)
- moved J1 128.3 mm to (63.0, 106.0)
- moved R6 127.6 mm to (65.4, 100.6), turned to 180 degrees
- moved L2 125.4 mm to (57.1, 88.4), turned to 90 degrees
- moved R8 125.3 mm to (58.7, 88.0), turned to 180 degrees
- moved C21 125.1 mm to (72.6, 91.3), turned to 90 degrees
- moved C11 124.8 mm to (69.0, 84.8), turned to 180 degrees
- moved C15 124.7 mm to (58.7, 88.8)
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Connections:
- U2 pad 22: /PC6 -> /PB14
- U2 pad 24: /PC6 -> /PB14
- U2 pad 26: /PC6 -> /PB14
- U6 pad 22: /PB14 -> /PC6
- U6 pad 24: /PB14 -> /PC6
- U6 pad 26: /PB14 -> /PC6
Routing:
- net /PB11_Rx3: track 0.00 -> 49.8 mm
- net /PA3_Rx2: track 0.00 -> 46.5 mm
- net /PB10_Tx3: track 0.00 -> 44.2 mm
- net /NRST: track 4.32 -> 43.1 mm, vias 0 -> 2
- net /PB14: track 5.28 -> 43.7 mm
- net /PA8_SCL: track 10.0 -> 39.5 mm
- net /PB15: track 6.85 -> 32.7 mm, vias 4 -> 3
- net /PB9: track 3.56 -> 28.7 mm, vias 1 -> 2
- net /PA14_SWCLK: track 0.00 -> 24.9 mm
- net /PB7: track 3.56 -> 26.1 mm, vias 1 -> 2
- net /PA13_SWDIO: track 0.00 -> 20.6 mm, vias 0 -> 2
- net /PB4: track 3.61 -> 24.2 mm
- net /PC11_SDA: track 8.41 -> 28.8 mm
- net /PB6: track 3.56 -> 24.0 mm, vias 1 -> 2
- net /PB8_BOOT0: track 3.71 -> 23.7 mm, vias 0 -> 2
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
Commit message: ...
Parts:
- added REF**: MountingHole_2.7mm, MountingHole:MountingHole_2.7mm, F.Cu at (141.6, 112.2)
- added REF**: MountingHole_2.7mm, MountingHole:MountingHole_2.7mm, F.Cu at (141.6, 68.3)
- added REF**: MountingHole_2.7mm, MountingHole:MountingHole_2.7mm, F.Cu at (97.8, 112.2)
- added REF**: MountingHole_2.7mm, MountingHole:MountingHole_2.7mm, F.Cu at (97.8, 68.3)
- moved JP6 61.6 mm to (114.8, 87.8), turned to 0 degrees
- moved JP4 59.2 mm to (114.8, 82.8)
- moved R24 59.0 mm to (126.4, 71.7)
- moved C20 58.0 mm to (138.8, 96.9)
- moved C35 58.0 mm to (128.3, 68.6)
- moved C6 58.0 mm to (131.1, 86.7)
- moved D5 58.0 mm to (131.5, 67.7)
- moved JP3 58.0 mm to (136.3, 92.9)
- moved R10 58.0 mm to (137.5, 100.6)
- moved R11 58.0 mm to (137.5, 99.6)
- moved R28 58.0 mm to (128.8, 67.1)
- moved C13 58.0 mm to (117.0, 95.3)
- moved C23 58.0 mm to (117.2, 96.9)
- moved C27 58.0 mm to (100.3, 91.8)
- moved C3 58.0 mm to (100.3, 79.6)
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Routing:
- net GND: track 79.4 -> 436.2 mm, vias 25 -> 39
- net +3V3: track 32.3 -> 279.7 mm, vias 2 -> 16
- net VCC: track 24.5 -> 210.4 mm
- net /FLT_DRV3: track 6.62 -> 26.9 mm, vias 0 -> 2
- net /PA11: track 0.00 -> 13.0 mm
- net /PA12: track 0.00 -> 13.0 mm
- net VBUS: track 1.87 -> 13.9 mm
- net /PA3_Rx2: track 46.5 -> 35.7 mm
- net /PA5: track 0.00 -> 10.6 mm
- net /PA6: track 0.00 -> 8.96 mm
- net /FLT_DRV2: track 8.38 -> 16.6 mm
- net /PA7: track 0.00 -> 7.00 mm
- net /PF0: track 1.67 -> 6.82 mm
- net /PB11_Rx3: track 49.8 -> 54.6 mm
- net /PB10_Tx3: track 44.2 -> 48.3 mm
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Other:
- board outline added: 50 x 50 mm

Commit message: ...
Parts:
- added G***: LOGO, Demo.preety:logosaola, F.Cu at (134.4, 82.7)
Connections:
- D2 pad 1: VCC -> +3V3
Routing:
- net GND: track 436.2 -> 522.3 mm, vias 39 -> 42
- net /PB2: track 2.06 -> 39.5 mm, vias 1 -> 5
- net +3V3: track 279.7 -> 300.1 mm
- net VCC: track 210.4 -> 190.7 mm
- net VBUS: track 13.9 -> 20.3 mm
- net /VDD33A: track 4.29 -> 9.22 mm
- net /PA8_SCL: track 39.5 -> 43.1 mm
- net /PB6: track 24.7 -> 28.0 mm
- net /PB7: track 26.3 -> 28.8 mm
- net /PB11_Rx3: track 54.6 -> 57.1 mm
- net /PB10_Tx3: track 48.3 -> 50.1 mm
- net /PB9: track 28.9 -> 30.5 mm
- net /PB4: track 24.2 -> 25.6 mm
- net /PC11_SDA: track 28.8 -> 30.1 mm
- net /PB8_BOOT0: track 25.3 -> 26.4 mm
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- added copper zone on B.Cu, net GND
