File: gimbal.kicad_sch (KiCad schematic)
At the start: 64 parts, among them J1 USB_C_Receptacle_USB2.0_16P, U1 STM32G431CBU6, U2 DRV8313PWP, U3 MPU-6050, U4 XC6206PxxxMR, U5 DRV8313PWP, U6 DRV8313PWP, Y1 Crystal, Y2 Crystal_GND23

Commit message: schematic
Parts:
- removed D3: LED, LED_SMD:LED_0603_1608Metric, symbol Device:LED
- removed JP1: SolderJumper_2_Open, Jumper:SolderJumper-2_P1.3mm_Bridged_RoundedPad1.0x1.5mm, symbol Jumper:SolderJumper_2_Open
- removed R9: 1K, symbol Device:R
- removed U4: XC6206PxxxMR, Package_TO_SOT_SMD:SOT-23-3, symbol Regulator_Linear:XC6206PxxxMR
- added C30: 0.01uF, Capacitor_SMD:C_01005_0402Metric, symbol Device:C
- added C31: 0.1uF, Capacitor_SMD:C_01005_0402Metric, symbol Device:C
- added C32: 10uF, Capacitor_SMD:C_01005_0402Metric, symbol Device:C
- added C33: 220pF, Capacitor_SMD:C_01005_0402Metric, symbol Device:C
- added C34: NS, Capacitor_SMD:C_01005_0402Metric, symbol Device:C
- added C35: 22uF, Capacitor_SMD:C_01005_0402Metric, symbol Device:C
- added C36, C37: 100nF, Capacitor_SMD:C_01005_0402Metric, symbol Device:C
- added C38, C39, C40: 4.7uF, Capacitor_SMD:C_01005_0402Metric, symbol Device:C
- added D6, D7: LED, LED_SMD:LED_0603_1608Metric, symbol Device:LED
- added D8: SS14, Diode_SMD:D_SMA, symbol Diode:SS14
- added D9: SMBJ15A, SMBJ15A:DIOM4336X265N, symbol SMBJ15A:SMBJ15A
- added J2: JTAG, Connector_PinHeader_1.00mm:PinHeader_1x04_P1.00mm_Vertical, symbol Connector_Generic:Conn_01x04
- added J3: Pitch, Connector_PinHeader_1.00mm:PinHeader_1x03_P1.00mm_Vertical, symbol Connector_Generic:Conn_01x03
- added J4: Roll, Connector_PinHeader_1.00mm:PinHeader_1x03_P1.00mm_Vertical, symbol Connector_Generic:Conn_01x03
- added J5: Yaw, Connector_PinHeader_1.00mm:PinHeader_1x03_P1.00mm_Vertical, symbol Connector_Generic:Conn_01x03
- added J6: IMU_Payload, Connector_PinHeader_1.00mm:PinHeader_1x04_P1.00mm_Vertical, symbol Connector_Generic:Conn_01x04
- added J7: Power_9V, Connector_AMASS:AMASS_XT30PW-M_1x02_P2.50mm_Horizontal, symbol Connector_Generic:Conn_01x02
- added J8: UART3, Connector_JST:JST_GH_BM04B-GHS-TBT_1x04-1MP_P1.25mm_Vertical, symbol Connector_Generic:Conn_01x04
- added J9: UART2, Connector_JST:JST_GH_BM04B-GHS-TBT_1x04-1MP_P1.25mm_Vertical, symbol Connector_Generic:Conn_01x04
- added JP3: SolderJumper_2_Open, Jumper:SolderJumper-2_P1.3mm_Bridged_RoundedPad1.0x1.5mm, symbol Jumper:SolderJumper_2_Open
- added JP4, JP5, JP6: (no value), Jumper:SolderJumper-2_P1.3mm_Bridged_RoundedPad1.0x1.5mm, symbol Jumper:SolderJumper_2_Open
- added L1: 10uH, Inductor_SMD:L_7.3x7.3_H3.5, symbol Device:L
- added L3: L_Ferrite, Inductor_SMD:L_0201_0603Metric, symbol Device:L_Ferrite
- added R19, R22: 330, Resistor_SMD:R_01005_0402Metric, symbol Device:R
- added R20, R21: 10k, Resistor_SMD:R_01005_0402Metric, symbol Device:R
- added R23: 100k, Resistor_SMD:R_01005_0402Metric, symbol Device:R
- added R24: 24.9k, Resistor_SMD:R_01005_0402Metric, symbol Device:R
- added R25: 200k, Resistor_SMD:R_01005_0402Metric, symbol Device:R
- added R26: 68.1k, Resistor_SMD:R_01005_0402Metric, symbol Device:R
- added R27, R29: 40.2k, Resistor_SMD:R_01005_0402Metric, symbol Device:R
- added R28: 124k, Resistor_SMD:R_01005_0402Metric, symbol Device:R
- added SW1, SW2: SW_Push, Button_Switch_THT:SW_PUSH_6mm_H5mm, symbol Switch:SW_Push
- added U7: MP1584EN, MP1584EN:SOIC127P600X170-9N, symbol MP1584EN:MP1584EN
- C1, C10, C11, C12, C13, C14, C15, C16, C17, C18, C19, C2, C20, C21, C25, C27, C29, C3, C4, C5, C6, C7, C8, C9: footprint (none) -> Capacitor_SMD:C_01005_0402Metric
- C22: value 0.47uF -> 100nF; footprint (none) -> Capacitor_SMD:C_01005_0402Metric
- C23: value 0.1uF -> 100nF; footprint (none) -> Capacitor_SMD:C_01005_0402Metric
- C24, C28: value 0.01uF -> 0.47uF; footprint (none) -> Capacitor_SMD:C_01005_0402Metric
- C26: value 0.47uF -> 0.01uF; footprint (none) -> Capacitor_SMD:C_01005_0402Metric
- J1: footprint (none) -> Connector_USB:USB_C_Receptacle_GCT_USB4105-xx-A_16P_TopMnt_Horizontal
- L2: footprint (none) -> Inductor_SMD:L_0402_1005Metric
- R1, R10, R11, R12, R16, R17, R2, R3, R4, R5, R6, R7, R8: footprint (none) -> Resistor_SMD:R_01005_0402Metric
- R13, R14: value 10k -> 5.1k; footprint (none) -> Resistor_SMD:R_01005_0402Metric
- R15, R18: value 330 -> 10k; footprint (none) -> Resistor_SMD:R_01005_0402Metric
Connections:
- net EN is gone; now on net PC6: U2.22 (EN3), U2.24 (EN2), U2.26 (EN1), U5.22 (EN3), U5.24 (EN2), U5.26 (EN1), U6.22 (EN3), U6.24 (EN2), U6.26 (EN1)
- net PA8 is gone; now on net PA8_SCL: U1.30 (PA8)
- net PC11 is gone; now on net PC11_SDA: U1.40 (PC11)
- net VBAT is gone; now on net +3V3: U1.1 (VBAT)
- net +3V3: now also C16.1, C23.2, R14.2, R15.1, R18.1, C35.1, J2.1 (Pin_1), J6.1 (Pin_1), J8.1 (Pin_1), J9.1 (Pin_1), L1.2, L3.1, R19.2, R20.1, R21.1, R22.2, R28.2, SW2.2; no longer R13.1, R14.1, R15.2, R16.1, R18.2
- net GND: now also C10.1, C11.1, C12.1, C13.1, C14.1, C15.1, C22.1, C23.1, C24.2, C27.2, C28.2, D4.1 (K), D5.1 (K), R16.2, C31.2, C32.2, C34.2, C35.2, C37.2, C38.2, C39.2, C40.2, D8.2 (A), D9.A, J2.4 (Pin_4), J6.4 (Pin_4), J7.1 (Pin_1), J8.4 (Pin_4), J9.4 (Pin_4), R24.2, R25.2, R26.2, R27.2, R29.2, SW1.1, U7.5 (GND), U7.9 (GND); no longer C22.2, C25.2, C26.2, C29.2
- net PA0: no longer U5.27 (IN1), U6.27 (IN1)
- net PA1: no longer U5.25 (IN2), U6.25 (IN2)
- net PA2: no longer U5.23 (IN3), U6.23 (IN3)
- net PA4: now also U5.25 (IN2)
- net PA5: now also JP4.2 (B)
- net PA6: now also JP5.2 (B)
- net PA7: now also JP6.2 (B)
- net PB0: now also U5.23 (IN3)
- net PB4: now also U5.27 (IN1)
- net PB6: now also U6.27 (IN1)
- net PB7: now also U6.25 (IN2)
- net PB9: now also U6.23 (IN3)
- net PC6: now also R13.1
- net Pitch1: now also J3.1 (Pin_1); no longer U5.5 (OUT1), U6.5 (OUT1)
- net Pitch2: now also J3.2 (Pin_2); no longer U5.8 (OUT2), U6.8 (OUT2)
- net Pitch3: now also J3.3 (Pin_3); no longer U5.9 (OUT3), U6.9 (OUT3)
- net VCC: now also C25.2, C27.1, C29.2, C31.1, C32.1, C37.1, C38.1, C39.1, C40.1, D9.C, J7.2 (Pin_2), R23.1, U7.7 (VIN); no longer C16.1, C23.2, C25.1, C27.2, C29.1
- net at U6.1 (CPL): now also C30.1; no longer C28.1
- net at U6.2 (CPH): now also C30.2; no longer C28.2
- net at C17.1, C18.1, R10.1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: now also L3.2
- net PC11_SDA: now reaches R10.2, U3.24 (SDA)
- net PC11_SDA: now also J6.3 (Pin_3)
- net at D4.2 (A): now also R13.2; no longer R15.1
- net at U5.1 (CPL): now also C26.1; no longer C24.1
- net at U5.2 (CPH): now also C26.2; no longer C24.2
- net PA8_SCL: now reaches R11.2, U3.23 (SCL)
- net PA8_SCL: now also J6.2 (Pin_2)
- net at U5.3 (VCP): now also C25.1; no longer C23.1
- net at U6.15 (V3P3): now also C28.1; no longer C26.1
- net at D5.2 (A): now also R14.1; no longer R18.1
- net at U5.15 (V3P3): now also C24.1; no longer C22.1
- net at U6.3 (VCP): now also C29.1; no longer C27.1
- removed net FLT_DRV: D1.1 (K), D4.1 (K), D5.1 (K), U2.18 (~{FAULT}), U5.18 (~{FAULT}), U6.18 (~{FAULT})
- net PA13 renamed PA13_SWDIO
- net PA13_SWDIO: now also J2.3 (Pin_3)
- net PA14 renamed PA14_SWCLK
- net PA14_SWCLK: now also J2.2 (Pin_2), JP3.1 (A)
- net PA3 renamed PA3_Rx2
- net PA3_Rx2: now also J9.3 (Pin_3)
- net PB10 renamed PB10_Tx3
- net PB10_Tx3: now also J8.2 (Pin_2)
- net PB11 renamed PB11_Rx3
- net PB11_Rx3: now also J8.3 (Pin_3)
- net PB8 renamed PB8_BOOT0
- net PB8_BOOT0: now also R16.1, SW2.1
- net PG10 renamed NRST
- net NRST: now also C22.2, R15.2, SW1.2
- removed net RST_DRV: R13.2, R16.2, R2.2, U2.16 (~{RESET}), U5.16 (~{RESET}), U6.16 (~{RESET})
- removed net SLP_DRV: R14.2, R17.2, R3.2, U2.17 (~{SLEEP}), U5.17 (~{SLEEP}), U6.17 (~{SLEEP})
- new net: R23.2, R24.1, U7.2 (EN)
- new net: R27.1, R28.1, R29.1, U7.4 (FB)
- new net: D7.2 (A), R22.1
- new net: C36.1, D8.1 (K), L1.1, U7.1 (SW)
- new net: C33.1, C34.1, U7.3 (COMP)
- new net: R25.1, U7.6 (FREQ)
- new net: C36.2, U7.8 (BST)
- new net: D6.2 (A), R19.1
- new net: C33.2, R26.1
- new net FLT_DRV1: D1.1 (K), JP4.1 (A), U2.18 (~{FAULT})
- new net FLT_DRV2: D6.1 (K), JP5.1 (A), U5.18 (~{FAULT})
- new net FLT_DRV3: D7.1 (K), JP6.1 (A), U6.18 (~{FAULT})
- new net PA14_Tx2: J9.2 (Pin_2), JP3.2 (B)
- new net RST_DRV1: R2.2, U2.16 (~{RESET})
- new net RST_DRV2: R17.2, U5.16 (~{RESET})
- new net RST_DRV3: R20.2, U6.16 (~{RESET})
- new net Roll1: J4.1 (Pin_1), U5.5 (OUT1)
- new net Roll2: J4.2 (Pin_2), U5.8 (OUT2)
- new net Roll3: J4.3 (Pin_3), U5.9 (OUT3)
- new net SLP_DRV1: R3.2, U2.17 (~{SLEEP})
- new net SLP_DRV2: R18.2, U5.17 (~{SLEEP})
- new net SLP_DRV3: R21.2, U6.17 (~{SLEEP})
- new net Yaw1: J5.1 (Pin_1), U6.5 (OUT1)
- new net Yaw2: J5.2 (Pin_2), U6.8 (OUT2)
- new net Yaw3: J5.3 (Pin_3), U6.9 (OUT3)
Other:
- note added: "FOC DRIVER"
- note added: "HEADER"
- note added: "IMU_FRAME"
- note added: "MCU"
- note added: "POWER"
- note added: "USB TYPE C"
- moved on the sheet: C1, C10, C11, C12, C13, C14, C15, C16, C17, C18, C19, C2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

Commit message: ...
Parts:
- SW1: value SW_Push -> Reset; footprint Button_Switch_THT:SW_PUSH_6mm_H5mm -> Button_Switch_SMD:SW_SPST_B3U-1000P
- SW2: value SW_Push -> Boot; footprint Button_Switch_THT:SW_PUSH_6mm_H5mm -> Button_Switch_SMD:SW_SPST_B3U-1000P
- Y1: footprint Crystal:Crystal_SMD_0603-2Pin_6.0x3.5mm_HandSoldering -> Crystal:Crystal_SMD_2012-2Pin_2.0x1.2mm_HandSoldering
- Y2: footprint Crystal:Crystal_SMD_3225-4Pin_3.2x2.5mm -> Crystal:Crystal_SMD_2016-4Pin_2.0x1.6mm
Other:
- moved on the sheet: C16, C17, C18, C19, C20, C21, C27, C28, C29, C3, C30, C31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
