File: gimbal.kicad_sch (KiCad schematic)
At the start: 103 parts, among them J1 USB_C_Receptacle_USB2.0_16P, J2 JTAG, J3 Pitch, J4 Roll, J5 Yaw, J6 IMU_Payload, J7 Power_9V, J8 UART3, J9 UART2, SW1 Reset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

Commit message: ...
Connections:
- net PB14: now also U6.22 (EN3), U6.24 (EN2), U6.26 (EN1)
- net PB15: now also U5.22 (EN3), U5.24 (EN2), U5.26 (EN1)
- net PC6: no longer U5.22 (EN3), U5.24 (EN2), U5.26 (EN1), U6.22 (EN3), U6.24 (EN2), U6.26 (EN1)
Changed lines of the file:
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@@
 		)
 	)
-	(label "PC6"
+	(label "PB15"
 		(at 161.29 171.45 0)
 		(effects
@@
 		)
 	)
-	(label "PC6"
+	(label "PB14"
 		(at 283.21 171.45 0)
 		(effects

Commit message: ...
Parts:
- removed D4: LED, LED_SMD:LED_0603_1608Metric, symbol Device:LED
- removed R13: 5.1k, Resistor_SMD:R_0201_0603Metric_Pad0.64x0.40mm_HandSolder, symbol Device:R
Connections:
- net PB14: now also U2.22 (EN3), U2.24 (EN2), U2.26 (EN1); no longer U6.22 (EN3), U6.24 (EN2), U6.26 (EN1)
- net PC6: now also U6.22 (EN3), U6.24 (EN2), U6.26 (EN1); no longer U2.22 (EN3), U2.24 (EN2), U2.26 (EN1)

Commit message: ...
Parts:
- J1: footprint Connector_USB:USB_C_Receptacle_GCT_USB4105-xx-A_16P_TopMnt_Horizontal -> Connector_USB:USB_C_Receptacle_GCT_USB4110
Connections:
- net +3V3: now also D2.1 (K)
- net VCC: no longer D2.1 (K)
Changed lines of the file:
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@@
 	(wire
 		(pts
+			(xy 349.25 38.1) (xy 349.25 44.45)
+		)
+		(stroke
+			(width 0)
+			(type default)
+		)
+	)
+	(wire
+		(pts
 			(xy 90.17 204.47) (xy 92.71 204.47)
 		)
@@
 	(wire
 		(pts
-			(xy 349.25 40.64) (xy 349.25 44.45)
-		)
-		(stroke
-			(width 0)
-			(type default)
-		)
-	)
-	(wire
-		(pts
 			(xy 119.38 102.87) (xy 119.38 111.76)
 		)
@@
 			)
 		)
-		(property "Footprint" "Connector_USB:USB_C_Receptacle_GCT_USB4105-xx-A_16P_TopMnt_Horizontal"
+		(property "Footprint" "Connector_USB:USB_C_Receptacle_GCT_USB4110"
 			(at 320.04 31.75 0)
 			(hide yes)
@@
 	)
 	(symbol
+		(lib_id "power:+3V3")
+		(at 349.25 38.1 0)
+		(unit 1)
+		(body_style 1)
+		(exclude_from_sim no)
+		(in_bom yes)
+		(on_board yes)
+		(in_pos_files yes)
+		(dnp no)
+		(property "Reference" "#PWR065"
+			(at 349.25 41.91 0)
+			(hide yes)
+			(show_name no)
+			(do_not_autoplace no)
+			(effects
+				(font
+					(size 1.27 1.27)
+				)
+			)
+		)
+		(property "Value" "+3V3"
+			(at 348.996 34.036 0)
+			(show_name no)
+			(do_not_autoplace no)
+			(effects
+				(font
+					(size 1.27 1.27)
+				)
+			)
+		)
+		(property "Footprint" ""
+			(at 349.25 38.1 0)
+			(hide yes)
+			(show_name no)
+			(do_not_autoplace no)
+			(effects
+				(font
+					(size 1.27 1.27)
+				)
+			)
+		)
+		(property "Datasheet" ""
+			(at 349.25 38.1 0)
+			(hide yes)
+			(show_name no)
+			(do_not_autoplace no)
+			(effects
+				(font
+					(size 1.27 1.27)
+				)
+			)
+		)
+		(property "Description" "Power symbol creates a global label with name \"+3V3\""
+			(at 349.25 38.1 0)
+			(hide yes)
+			(show_name no)
+			(do_not_autoplace no)
+			(effects
+				(font
+					(size 1.27 1.27)
+				)
+			)
+		)
+		(pin "1"
+		)
+		(instances
+			(project "gimbal"
+				(path "/3eb7d9fe-c3b4-4b53-9f23-9f8dbb8724ef"
+					(reference "#PWR065")
+					(unit 1)
+				)
+			)
+		)
+	)
+	(symbol
 		(lib_id "Device:R")
 		(at 303.53 87.63 0)
@@
 					(unit 1)
 				)
-			)
-		)
-	)
-	(symbol
-		(lib_id "power:VCC")
-		(at 349.25 40.64 0)
-		(unit 1)
-		(body_style 1)
-		(exclude_from_sim no)
-		(in_bom yes)
-		(on_board yes)
-		(in_pos_files yes)
-		(dnp no)
-		(fields_autoplaced yes)
-		(property "Reference" "#PWR013"
-			(at 349.25 44.45 0)
-			(hide yes)
-			(show_name no)
-			(do_not_autoplace no)
-			(effects
-				(font
-					(size 1.27 1.27)
-				)
-			)
-		)
-		(property "Value" "VCC"
-			(at 349.25 35.56 0)
-			(show_name no)
-			(do_not_autoplace no)
-			(effects
-				(font
-					(size 1.27 1.27)
-				)
-			)
-		)
-		(property "Footprint" ""
-			(at 349.25 40.64 0)
-			(hide yes)
-			(show_name no)
-			(do_not_autoplace no)
-			(effects
-				(font
-					(size 1.27 1.27)
-				)
-			)
-		)
-		(property "Datasheet" ""
-			(at 349.25 40.64 0)
-			(hide yes)
-			(show_name no)
-			(do_not_autoplace no)
-			(effects
-				(font
-					(size 1.27 1.27)
-				)
-			)
-		)
-		(property "Description" "Power symbol creates a global label with name \"VCC\""
-			(at 349.25 40.64 0)
-			(hide yes)
-			(show_name no)
-			(do_not_autoplace no)
-			(effects
-				(font
-					(size 1.27 1.27)
-				)
-			)
-		)
-		(pin "1"
-		)
-		(instances
-			(project "gimbal"
-				(path "/3eb7d9fe-c3b4-4b53-9f23-9f8dbb8724ef"
-					(reference "#PWR013")
-					(unit 1)
-				)
