File: recovery/gimbal_recovered.kicad_pcb (KiCad board)
At the start: 2 copper layers, 103 parts, among them J1 USB_C_Receptacle_USB2.0_16P, J2 JTAG, J3 Pitch, J4 Roll, J5 Yaw, J6 IMU_Payload, J7 Power_9V, J8 UART3, J9 UART2, SW1 Reset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

Commit message: ...
Parts:
- J7: footprint Connector_AMASS:AMASS_XT30U-F_1x02_P5.0mm_Vertical -> Connector_AMASS:AMASS_XT30PW-M_1x02_P2.50mm_Horizontal
- moved J2 71.7 mm to (119.0, 149.8)
- moved C19 54.5 mm to (140.0, 147.8), turned to -90 degrees
- moved C18 54.4 mm to (141.6, 147.2), turned to 180 degrees
- moved L3 54.1 mm to (143.7, 146.2), turned to 180 degrees
- moved R12 54.0 mm to (139.1, 147.8), turned to -90 degrees
- moved C20 53.5 mm to (138.1, 147.8), turned to -90 degrees
- moved C16 51.7 mm to (144.0, 144.8), turned to 90 degrees
- moved C17 50.8 mm to (143.0, 144.8), turned to 90 degrees
- moved R13 48.7 mm to (140.3, 157.4), turned to 90 degrees
- moved D4 47.9 mm to (141.5, 158.2)
- moved SW2 47.9 mm to (140.5, 163.6)
- moved R16 47.9 mm to (138.2, 162.1)
- moved C10 47.5 mm to (124.6, 148.0)
- moved C11 47.5 mm to (134.3, 141.5)
- moved C12 47.5 mm to (131.8, 149.9)
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Routing:
- net GND: track 19.5 -> 0.00 mm
- net +3V3: track 10.8 -> 0.00 mm
- net VCC: track 7.70 -> 0.00 mm
- net /Yaw1: track 6.87 -> 0.00 mm
- net /Yaw3: track 6.51 -> 0.00 mm
- net /Yaw2: track 6.07 -> 0.00 mm
- net /FLT_DRV3: track 5.62 -> 0.00 mm
- net Net-(U3-VDD): track 5.54 -> 0.00 mm
- net /VDD33A: track 5.25 -> 0.00 mm
- net /NRST: track 4.32 -> 0.00 mm
- net /PB8_BOOT0: track 3.71 -> 0.00 mm
- net /VREF: track 3.10 -> 0.00 mm
- net Net-(U6-V3P3): track 2.29 -> 0.00 mm
- net /RST_DRV3: track 2.15 -> 0.00 mm
- net /SLP_DRV3: track 2.01 -> 0.00 mm
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