File: recovery/gimbal_recovered.kicad_sch (KiCad schematic)
At the start: 103 parts, among them J1 USB_C_Receptacle_USB2.0_16P, J2 JTAG, J3 Pitch, J4 Roll, J5 Yaw, J6 IMU_Payload, J7 Power_9V, J8 UART3, J9 UART2, SW1 Reset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

Commit message: ...
Parts:
- J7: footprint Connector_AMASS:AMASS_XT30U-F_1x02_P5.0mm_Vertical -> Connector_AMASS:AMASS_XT30PW-M_1x02_P2.50mm_Horizontal
Changed lines of the file:
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@@
 			)
 		)
-		(property "Footprint" "Connector_AMASS:AMASS_XT30U-F_1x02_P5.0mm_Vertical"
+		(property "Footprint" "Connector_AMASS:AMASS_XT30PW-M_1x02_P2.50mm_Horizontal"
 			(at 91.44 273.05 0)
 			(hide yes)
